File: flf.kicad_sch (KiCad schematic)
At the start: 24 parts, among them J1 Conn_01x04_Pin, J2 XT30UPB-M, U1 STM32F411CCUx, U2 TPS563208DDCR, U3 MAX14870ETC_T, Y1 Crystal

Commit message: Updated schematic
Parts:
- removed D2: LED, symbol Device:LED
- removed L1: 2.2u, symbol Device:L_Small
- removed U1: STM32F411CCUx, Package_DFN_QFN:QFN-48-1EP_7x7mm_P0.5mm_EP5.6x5.6mm, symbol MCU_ST_STM32F4:STM32F411CCUx
- removed U2: TPS563208DDCR, TPS563208DDCR:SOT95P280X110-6N, symbol customs:TPS563208DDCR
- removed U3: MAX14870ETC_T, MAX14870ETC_T:SON50P300X300X80-13N, symbol customs:MAX14870ETC_T
- added C11, C18, C19, C20, C21, C22, C23: 0.1u, symbol Device:C_Small
- added C12, C13, C15, C16: 10u, symbol Device:C_Small
- added C14, C17: 100n, symbol Device:C_Small
- added IC1: TB6612FNG, TB6612FNG:SSOP24, symbol customs:TB6612FNG
- added J3, J4: Conn_01x02_Socket, symbol Connector:Conn_01x02_Socket
- added M1, M2: ~, symbol customs:n20_motor
- added MM1, MM2: ~, symbol customs:motor_mounts
- added MP1: ~, symbol customs:MP1584
- added R10, R12, R16, R18, R19, R20, R9: 220, symbol Device:R_Small
- added R11, R13, R14, R15, R17, R21, R22, R23: 100, symbol Device:R_Small
- added R5, R7, R8: 10k, symbol Device:R
- added R6: 3.3k, symbol Device:R
- added U1: STM32F411CEUx, Package_DFN_QFN:QFN-48-1EP_7x7mm_P0.5mm_EP5.6x5.6mm, symbol MCU_ST_STM32F4:STM32F411CEUx
- added U10, U11, U3, U4, U5, U6, U7, U8, U9: QRE1113GR, QRE1113GR:SOIC180P460X187-4N, symbol customs:QRE1113GR
- added U2: TCRT5000L, TCRT5000L:XDCR_TCRT5000L, symbol customs:TCRT5000L
- C10: value 22u -> 0.1u
- C6, C7: value 100n -> 33p
- C8: value 10u -> 22u
- C9: value 100n -> 0.1u
- R1: value R -> 1k
- R2, R4: value 33.2k -> 220
- R3: value 10k -> 100
Connections:
- net +3.3V: now also C10.2, C8.2, C9.2, R3.2, C11.2, C14.1, C15.1, C18.2, C19.2, C20.2, C21.2, C22.2, C23.2, IC1.19 (STBY), IC1.20 (VCC), MP1. (IN+), R11.2, R13.2, R14.2, R15.2, R17.2, R21.2, R22.2, R23.2, R8.2, U1.1 (VBAT), U1.24 (VDD), U1.36 (VDD), U1.48 (VDD)
- net BAT+: now also C16.1, C17.1, IC1.13 (VM2), IC1.14 (VM3), IC1.24 (VM1), MP1. (IN+), R5.2; no longer C8.1
- net GND: now also C8.1, C12.2, C13.1, C14.2, C15.2, C16.2, C17.2, IC1.18 (GND), MP1. (IN+), R6.1, R7.2, U10.2, U10.4, U11.2, U11.4, U3.2, U3.4, U4.2, U4.4, U5.2, U5.4, U6.2, U6.4, U7.2, U7.4, U8.2, U8.4, U9.2, U9.4; no longer C10.2, C8.2, J2.N, R3.2
- net LED: now also U1.2 (PC13)
- net OSC_IN: now also U1.5 (PH0)
- net OSC_OUT: now also U1.6 (PH1)
- net VDDA: now also U1.9 (VDDA)
- net Pin: now reaches R4.1
- net Pin: now also R2.1, R10.1, R12.1, R16.1, R18.1, R19.1, R20.1, R9.1
- net at C9.1: now also R2.2, U4.3
- net at C10.1, R4.2: now also U3.3; no longer R2.2
- net at R3.1: now also U4.1; no longer R2.1
- new net: R21.1, U9.1
- new net: C18.1, R9.2, U5.3
- new net: U1.23 (VSS), U1.35 (VSS), U1.47 (VSS), U1.49 (VSS)
- new net: C21.1, R18.2, U9.3
- new net: C19.1, R10.2, U7.3
- new net: R22.1, U10.1
- new net: R11.1, U3.1
- new net: R15.1, U7.1
- new net: R13.1, U6.1
- new net: C22.1, R19.2, U10.3
- new net: R23.1, U11.1
- new net: C11.1, R12.2, U6.3
- new net: C23.1, R20.2, U11.3
- new net: C20.1, R16.2, U8.3
- new net: R14.1, U5.1
- new net: R17.1, U8.1
- new net BAT-: IC1.10 (PGND2'), IC1.3 (PGND1), IC1.4 (PGND1'), IC1.9 (PGND2), J2.N, MP1. (IN+)
- new net BAT_SNS: C13.2, R5.1, R6.2
- new net M1_IN1: IC1.21 (AIN1)
- new net M1_IN2: IC1.22 (AIN2)
- new net M1_PWM: IC1.23 (PWMA)
- new net M2_IN1: IC1.17 (BIN1)
- new net M2_IN2: IC1.16 (BIN2)
- new net M2_PWM: IC1.15 (PWMB)
- new net Motor1+: IC1.1 (AO1), IC1.2 (AO1'), J3.1 (Pin_1)
- new net Motor1-: IC1.5 (AO2), IC1.6 (AO2'), J3.2 (Pin_2)
- new net Motor2+: IC1.7 (BO2), IC1.8 (BO2'), J4.1 (Pin_1)
- new net Motor2-: IC1.11 (BO1), IC1.12 (BO1'), J4.2 (Pin_2)
- new net Pull D: R7.1, U1.44 (BOOT0)
- new net Pull U: R8.1, U1.7 (NRST)
- new net VCAP: C12.1, U1.22 (VCAP1)
Other:
- note added: "Battery"
- note added: "Decoupling capacitors"
- note added: "MCU"
- note added: "MCU connections"
- note added: "Microbuck"
- note added: "Motor Driver"
- note added: "Motor components"
- note added: "Motor connectors"
- note added: "Motor mounts"
- note added: "Motors"
- note added: "Oscillator"
- note added: "Power"
- note added: "QRE1113 Sensors"
- note added: "Serial Wire"
- moved on the sheet: C1, C2, C3, C4, C5, C6, C7, D1, FB1, J1, J2, R1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
