File: Lavender 1.0/untitled.kicad_sch (KiCad schematic)
At the start: 72 parts, among them U10 QRE1113GR, U11 QRE1113GR, U12 QRE1113GR, U13 QRE1113GR, U14 QRE1113GR, U15 QRE1113GR, U16 QRE1113GR, U17 QRE1113GR, U18 QRE1113GR, U19 TCRT5000L, U2 TCRT5000L, U20 TCRT5000L, U4 TCRT5000L, U5 TCRT5000L, U6 TCRT5000L, U7 TCRT5000L, U8 TCRT5000L, U9 TCRT5000L

Commit message: arrange pcb components
Parts:
- R19, R20, R21, R22, R23, R24, R25, R26, R27, R28, R29, R30, R31, R32, R33, R34, R35, R36, R37, R38, R39, R40, R41, R42, R43, R44, R45, R49, R50, R51, R52, R53, R54, R55, R56, R57, R58, R59, R60, R61, R62, R63, R64, R65, R66, R67, R68, R69, R70, R71, R72, R73, R74, R75: footprint (none) -> Resistor_SMD:R_0603_1608Metric_Pad0.98x0.95mm_HandSolder
- U10, U11, U12, U13, U14, U15, U16, U17, U18: footprint QRE1113GR:SOIC180P460X187-4N -> customs:QRE1113-SMD
- U19, U2, U20, U4, U5, U6, U7, U8, U9: footprint TCRT5000L:XDCR_TCRT5000L -> customs:XDCR_TCRT5000L

Commit message: started routing
Parts:
- added R46, R47, R48, R82, R85, R88, R91: 150, Resistor_SMD:R_0603_1608Metric_Pad0.98x0.95mm_HandSolder, symbol Device:R_Small
- added R76, R77, R78, R83, R86, R89, R92: 4k7, Resistor_SMD:R_0603_1608Metric_Pad0.98x0.95mm_HandSolder, symbol Device:R_Small
- added R79, R80, R81, R84, R87, R90, R93: 220, Resistor_SMD:R_0603_1608Metric_Pad0.98x0.95mm_HandSolder, symbol Device:R_Small
- added U21, U22, U23, U24, U25, U26, U27: QRE1113GR, customs:QRE1113-SMD, symbol customs:QRE1113GR
Connections:
- net T_PWR is gone; now on net +3.3V: R49.1, R50.1, R52.1, R53.1, R55.1, R56.1, R58.1, R59.1, R61.1, R62.1, R64.1, R65.1, R67.1, R68.1, R70.1, R71.1, R73.1, R74.1
- net GND: now also U21.2, U21.4, U22.2, U22.4, U23.2, U23.4, U24.2, U24.4, U25.2, U25.4, U26.2, U26.4, U27.2, U27.4
- net Q4: now also R79.1; no longer R30.1
- net Q5: now also R30.1; no longer R33.1
- net Q6: now also R33.1; no longer R36.1
- net Q7: now also R36.1; no longer R39.1
- net Q8: now also R80.1; no longer R42.1
- net Q9: now also R39.1; no longer R45.1
- net Q_PWR renamed +3.3V
- net +3.3V: now also R46.2, R47.2, R48.2, R76.2, R77.2, R78.2, R82.2, R83.2, R85.2, R86.2, R88.2, R89.2, R91.2, R92.2
- new net: R77.1, R80.2, U22.3
- new net: R46.1, U21.1
- new net: R76.1, R79.2, U21.3
- new net: R88.1, U26.1
- new net: R47.1, U22.1
- new net: R48.1, U23.1
- new net: R78.1, R81.2, U23.3
- new net: R89.1, R90.2, U26.3
- new net: R86.1, R87.2, U25.3
- new net: R91.1, U27.1
- new net: R92.1, R93.2, U27.3
- new net: R83.1, R84.2, U24.3
- new net: R85.1, U25.1
- new net: R82.1, U24.1
- new net Q10: R42.1
- new net Q11: R45.1
- new net Q12: R81.1
- new net Q13: R84.1
- new net Q14: R87.1
- new net Q15: R90.1
- new net Q16: R93.1

Commit message: Start third sensor array
Parts:
- removed R49, R52, R55, R58, R61, R64, R67, R70, R73: 150, Resistor_SMD:R_0603_1608Metric_Pad0.98x0.95mm_HandSolder, symbol Device:R_Small
- removed R50, R53, R56, R59, R62, R65, R68, R71, R74: 4k7, Resistor_SMD:R_0603_1608Metric_Pad0.98x0.95mm_HandSolder, symbol Device:R_Small
- removed R51, R54, R57, R60, R63, R66, R69, R72, R75: 220, Resistor_SMD:R_0603_1608Metric_Pad0.98x0.95mm_HandSolder, symbol Device:R_Small
- removed U19, U2, U20, U4, U5, U6, U7, U8, U9: TCRT5000L, customs:XDCR_TCRT5000L, symbol customs:TCRT5000L
- added R100, R101, R102, R109, R110, R111, R118, R119, R120: 220, Resistor_SMD:R_0603_1608Metric_Pad0.98x0.95mm_HandSolder, symbol Device:R_Small
- added R103, R104, R105, R112, R113, R114, R94, R95, R96: 150, Resistor_SMD:R_0603_1608Metric_Pad0.98x0.95mm_HandSolder, symbol Device:R_Small
- added R106, R107, R108, R115, R116, R117, R97, R98, R99: 4k7, Resistor_SMD:R_0603_1608Metric_Pad0.98x0.95mm_HandSolder, symbol Device:R_Small
- added U28, U29, U30, U31, U32, U33, U34, U35, U36: QRE1113GR, customs:QRE1113-SMD, symbol customs:QRE1113GR
Connections:
- net +3.3V: now also R103.2, R104.2, R105.2, R106.2, R107.2, R108.2, R112.2, R113.2, R114.2, R115.2, R116.2, R117.2, R94.2, R95.2, R96.2, R97.2, R98.2, R99.2
- net GND: now also U28.2, U28.4, U29.2, U29.4, U30.2, U30.4, U31.2, U31.4, U32.2, U32.4, U33.2, U33.4, U34.2, U34.4, U35.2, U35.4, U36.2, U36.4
- new net: R107.1, R110.2, U32.3
- new net: R117.1, R120.2, U36.3
- new net: R94.1, U28.1
- new net: R105.1, U33.1
- new net: R108.1, R111.2, U33.3
- new net: R101.2, R98.1, U29.3
- new net: R104.1, U32.1
- new net: R114.1, U36.1
- new net: R100.2, R97.1, U28.3
- new net: R106.1, R109.2, U31.3
- new net: R96.1, U30.1
- new net: R102.2, R99.1, U30.3
- new net: R116.1, R119.2, U35.3
- new net: R113.1, U35.1
- new net: R115.1, R118.2, U34.3
- new net: R112.1, U34.1
- new net: R95.1, U29.1
- new net: R103.1, U31.1
- new net N1: R100.1
- new net N2: R109.1
- new net N3: R118.1
- new net N4: R101.1
- new net N5: R110.1
- new net N6: R119.1
- new net N7: R102.1
- new net N8: R111.1
- new net N9: R120.1
Other:
- note added: "QRE1113 Sensors (9 sensor array)"
- note added: "QRE1113 Sensors(16 sensor array)"
- note removed: "QRE1113 Sensors"
- note removed: "TCRT5000L Sensors"
