File: Lavender 1.0/line follower simple.kicad_pcb (KiCad board)
At the start: 2 copper layers, 112 parts, among them J1 XT30UPB-M, J2 Conn_01x06_Socket, J5 Conn_01x06_Socket, J6 Conn_02x06_Counter_Clockwise, J7 Conn_02x06_Counter_Clockwise, SW2 SW_Push, SW5 SW_Push_DPDT, SW6 SW_Push_DPDT, U10 QRE1113GR, U11 QRE1113GR, U12 QRE1113GR, U13 QRE1113GR, U14 QRE1113GR, U15 QRE1113GR, U16 QRE1113GR, U17 QRE1113GR, U18 QRE1113GR, U19 TCRT5000L, U2 TCRT5000L, U20 TCRT5000L, U21 BNO055, U4 TCRT5000L, U5 TCRT5000L, U6 TCRT5000L, U7 TCRT5000L, U8 TCRT5000L, U9 TCRT5000L

Commit message: started routing
Parts:
- removed D1, D2: LED, LED_THT:LED_D5.0mm
- removed J6, J7: Conn_02x06_Counter_Clockwise, Connector_IDC:IDC-Header_2x06_P2.54mm_Vertical_SMD
- removed JP1, JP10, JP11, JP12, JP13, JP14, JP15, JP16, JP17, JP18, JP19, JP2, JP20, JP3, JP4, JP5, JP6, JP7, JP8, JP9: SolderJumper_2_Open, Jumper:SolderJumper-2_P1.3mm_Open_RoundedPad1.0x1.5mm
- removed R1, R2: 47, Resistor_SMD:R_0603_1608Metric_Pad0.98x0.95mm_HandSolder
- added H1: MountingHole, customs:2mm hole, F.Cu at (101.3, 117.6)
- added H2: MountingHole, customs:2mm hole, F.Cu at (120.2, 117.6)
- added H3: MountingHole, customs:2mm hole, F.Cu at (160.5, 111.6)
- added H4: MountingHole, customs:2mm hole, F.Cu at (163.5, 111.6)
- added J10: Conn_01x13_Pin, Connector_PinHeader_2.54mm:PinHeader_1x13_P2.54mm_Vertical, F.Cu at (75.8, 155.2)
- added J11: Conn_01x13_Pin, Connector_PinHeader_2.54mm:PinHeader_1x13_P2.54mm_Vertical, F.Cu at (144.4, 155.2)
- added J12: Conn_01x13_Pin, Connector_PinHeader_2.54mm:PinHeader_1x13_P2.54mm_Vertical, F.Cu at (190.7, 113.7)
- added J13: Conn_01x13_Pin, Connector_PinHeader_2.54mm:PinHeader_1x13_P2.54mm_Vertical, F.Cu at (259.2, 113.7)
- added J14: Conn_01x20, Connector_FFC-FPC:Amphenol_F32Q-1A7x1-11020_1x20-1MP_P0.5mm_Horizontal, F.Cu at (110.5, 81.4)
- added J15: Conn_01x20, Connector_FFC-FPC:Amphenol_F32Q-1A7x1-11020_1x20-1MP_P0.5mm_Horizontal, F.Cu at (110.0, 120.5)
- added J3: Conn_01x02_Pin, Connector_PinHeader_2.54mm:PinHeader_1x02_P2.54mm_Vertical, F.Cu at (72.1, 160.2)
- added J4: Conn_01x02_Pin, Connector_PinHeader_2.54mm:PinHeader_1x02_P2.54mm_Vertical, F.Cu at (148.1, 160.6)
- added J8: Conn_01x28_Pin, Connector_PinHeader_2.54mm:PinHeader_1x28_P2.54mm_Vertical, F.Cu at (75.8, 152.6)
- added R46: 150, Resistor_SMD:R_0603_1608Metric_Pad0.98x0.95mm_HandSolder, F.Cu at (66.2, 60.4)
- added R47: 150, Resistor_SMD:R_0603_1608Metric_Pad0.98x0.95mm_HandSolder, F.Cu at (104.8, 46.1)
- added R48: 150, Resistor_SMD:R_0603_1608Metric_Pad0.98x0.95mm_HandSolder, F.Cu at (146.5, 54.9)
- added R76: 4k7, Resistor_SMD:R_0603_1608Metric_Pad0.98x0.95mm_HandSolder, F.Cu at (66.2, 62.2)
- added R77: 4k7, Resistor_SMD:R_0603_1608Metric_Pad0.98x0.95mm_HandSolder, F.Cu at (104.8, 48.1)
- added R78: 4k7, Resistor_SMD:R_0603_1608Metric_Pad0.98x0.95mm_HandSolder, F.Cu at (146.6, 56.8)
- added R79: 220, Resistor_SMD:R_0603_1608Metric_Pad0.98x0.95mm_HandSolder, F.Cu at (66.9, 64.3)
- added R80: 220, Resistor_SMD:R_0603_1608Metric_Pad0.98x0.95mm_HandSolder, F.Cu at (106.1, 50.0)
- added R81: 220, Resistor_SMD:R_0603_1608Metric_Pad0.98x0.95mm_HandSolder, F.Cu at (144.8, 59.2)
- added R82: 150, Resistor_SMD:R_0603_1608Metric_Pad0.98x0.95mm_HandSolder, F.Cu at (156.3, 60.0)
- added R83: 4k7, Resistor_SMD:R_0603_1608Metric_Pad0.98x0.95mm_HandSolder, F.Cu at (156.3, 61.7)
- added R84: 220, Resistor_SMD:R_0603_1608Metric_Pad0.98x0.95mm_HandSolder, F.Cu at (154.7, 64.4)
- added R85: 150, Resistor_SMD:R_0603_1608Metric_Pad0.98x0.95mm_HandSolder, F.Cu at (165.0, 70.7)
- added R86: 4k7, Resistor_SMD:R_0603_1608Metric_Pad0.98x0.95mm_HandSolder, F.Cu at (165.0, 72.5)
- added R87: 220, Resistor_SMD:R_0603_1608Metric_Pad0.98x0.95mm_HandSolder, F.Cu at (163.4, 75.2)
- added R88: 150, Resistor_SMD:R_0603_1608Metric_Pad0.98x0.95mm_HandSolder, F.Cu at (170.3, 82.0)
- added R89: 4k7, Resistor_SMD:R_0603_1608Metric_Pad0.98x0.95mm_HandSolder, F.Cu at (170.4, 80.5)
- added R90: 220, Resistor_SMD:R_0603_1608Metric_Pad0.98x0.95mm_HandSolder, F.Cu at (168.8, 85.0)
- added R91: 150, Resistor_SMD:R_0603_1608Metric_Pad0.98x0.95mm_HandSolder, F.Cu at (171.9, 91.9)
- added R92: 4k7, Resistor_SMD:R_0603_1608Metric_Pad0.98x0.95mm_HandSolder, F.Cu at (171.8, 94.0)
- added R93: 220, Resistor_SMD:R_0603_1608Metric_Pad0.98x0.95mm_HandSolder, F.Cu at (169.4, 96.2)
- added U1: 74HC4067, customs:74HC4067-Mux, F.Cu at (110.7, 66.3)
- added U22: QRE1113GR, customs:QRE1113-SMD, B.Cu at (105.7, 48.1)
- added U23: QRE1113GR, customs:QRE1113-SMD, B.Cu at (145.7, 57.1)
- added U24: QRE1113GR, customs:QRE1113-SMD, B.Cu at (155.7, 62.2)
- added U25: QRE1113GR, customs:QRE1113-SMD, B.Cu at (164.7, 72.9)
- added U26: QRE1113GR, customs:QRE1113-SMD, B.Cu at (170.1, 82.8)
- added U27: QRE1113GR, customs:QRE1113-SMD, B.Cu at (171.4, 94.2)
- J1, R5, R6, U10, U11, U12, U13, U14, U15, U16, U17, U18: moved to B.Cu
- J2: value Conn_01x06_Socket -> Conn_01x20; footprint Connector_JST:JST_SH_BM06B-SRSS-TB_1x06-1MP_P1.00mm_Vertical -> Connector_FFC-FPC:Amphenol_F32Q-1A7x1-11020_1x20-1MP_P0.5mm_Horizontal
- J5: value Conn_01x06_Socket -> Conn_01x28_Pin; footprint Connector_JST:JST_SH_BM06B-SRSS-TB_1x06-1MP_P1.00mm_Vertical -> Connector_PinHeader_2.54mm:PinHeader_1x28_P2.54mm_Vertical
- U21: value BNO055 -> QRE1113GR; footprint customs:BNO055 module -> customs:QRE1113-SMD
- moved U18 171.3 mm to (135.7, 54.6), turned to 180 degrees
- moved U17 168.8 mm to (125.7, 48.1), turned to 180 degrees
- moved R43 168.5 mm to (136.1, 52.5), turned to 180 degrees
- moved R44 168.5 mm to (135.9, 54.5), turned to 180 degrees
- moved R45 166.9 mm to (134.2, 56.8)
- moved U16 164.3 mm to (115.7, 48.1), turned to 180 degrees
- moved R40 158.6 mm to (126.2, 46.0), turned to 180 degrees
- moved R41 158.6 mm to (126.0, 47.8), turned to 180 degrees
- moved R42 157.2 mm to (124.5, 50.0)
- moved R38 147.6 mm to (116.1, 48.0), turned to 180 degrees
- moved R37 147.4 mm to (116.0, 46.0), turned to 180 degrees
- moved R39 145.9 mm to (114.4, 50.2)
- moved R36 135.9 mm to (96.7, 50.6), turned to 180 degrees
- moved R35 134.6 mm to (95.3, 48.0)
- moved R34 134.2 mm to (95.2, 46.1)
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Connections:
- BlackPill1 pad 30: LED -> unconnected-(BlackPill1-PA15-Pad30)
- BlackPill1 pad 36: IMU_SCL -> unconnected-(BlackPill1-PB8-Pad36)
- BlackPill1 pad 37: IMU_SDA -> unconnected-(BlackPill1-PB9-Pad37)
- BlackPill1 pad 4: IMU_RST -> unconnected-(BlackPill1-PB10-Pad4)
- J2 pad 1: Motor1+ -> +3.3V
- J2 pad 2: GND -> T8
- J2 pad 3: M1_C1 -> GND
- J2 pad 4: M1_C2 -> T7
- J2 pad 5: +3.3V -> GND
- J2 pad 6: Motor1- -> T6
- J5 pad 1: Motor2+ -> GND
- J5 pad 3: M2_C1 -> PWMA_t
- J5 pad 4: M2_C2 -> AIN2_t
- J5 pad 5: +3.3V -> AIN1_t
- J5 pad 6: Motor2- -> GND
- R22 pad 2: Q_PWR -> +3.3V
- R23 pad 2: Q_PWR -> +3.3V
- R24 pad 2: Q_PWR -> +3.3V
- R25 pad 2: Q_PWR -> +3.3V
- R26 pad 2: Q_PWR -> +3.3V
- R27 pad 2: Q_PWR -> +3.3V
- R28 pad 2: Q_PWR -> +3.3V
- R29 pad 2: Q_PWR -> +3.3V
- R30 pad 1: Q4 -> Q5
- R31 pad 2: Q_PWR -> +3.3V
- R32 pad 2: Q_PWR -> +3.3V
- R33 pad 1: Q5 -> Q6
- R34 pad 2: Q_PWR -> +3.3V
- R35 pad 2: Q_PWR -> +3.3V
- R36 pad 1: Q6 -> Q7
- R37 pad 2: Q_PWR -> +3.3V
- R38 pad 2: Q_PWR -> +3.3V
- R39 pad 1: Q7 -> Q9
- R40 pad 2: Q_PWR -> +3.3V
- R41 pad 2: Q_PWR -> +3.3V
- R42 pad 1: Q8 -> Q10
- R43 pad 2: Q_PWR -> +3.3V
- R44 pad 2: Q_PWR -> +3.3V
- R45 pad 1: Q9 -> Q11
- R49 pad 1: T_PWR -> +3.3V
- R50 pad 1: T_PWR -> +3.3V
- R52 pad 1: T_PWR -> +3.3V
- R53 pad 1: T_PWR -> +3.3V
- R55 pad 1: T_PWR -> +3.3V
- R56 pad 1: T_PWR -> +3.3V
- R58 pad 1: T_PWR -> +3.3V
- R59 pad 1: T_PWR -> +3.3V
- R61 pad 1: T_PWR -> +3.3V
- R62 pad 1: T_PWR -> +3.3V
- R64 pad 1: T_PWR -> +3.3V
- R65 pad 1: T_PWR -> +3.3V
- R67 pad 1: T_PWR -> +3.3V
- R68 pad 1: T_PWR -> +3.3V
- R70 pad 1: T_PWR -> +3.3V
- R71 pad 1: T_PWR -> +3.3V
- R73 pad 1: T_PWR -> +3.3V
- R74 pad 1: T_PWR -> +3.3V
- SW5 pad 2: BAT+ -> BAT+_t
- SW5 pad 5: BAT+ -> BAT+_t
- TB1 pad 10: Motor2+ -> Motor2+_t
- TB1 pad 11: Motor2- -> Motor2-_t
- TB1 pad 12: Motor1- -> Motor1-_t
- TB1 pad 13: Motor1+ -> Motor1+_t
- TB1 pad 2: PWMB -> PWMB_t
- TB1 pad 3: BIN2 -> BIN2_t
- TB1 pad 4: BIN1 -> BIN1_t
- TB1 pad 6: AIN1 -> AIN1_t
- TB1 pad 7: AIN2 -> AIN2_t
- TB1 pad 8: PWMA -> PWMA_t
- U21 pad 1: +3.3V -> Net-(R46-Pad1)
- U21 pad 2: unconnected-(U21-3V3-Pad2) -> GND
- U21 pad 3: GND -> Net-(R76-Pad1)
- U21 pad 4: IMU_SDA -> GND
Routing:
- net +3.3V: track 0.00 -> 211.7 mm, vias 0 -> 3
- net BAT_SNS: track 0.00 -> 56.5 mm
- net BAT+_out: track 0.00 -> 54.3 mm
- net EN: track 0.00 -> 53.0 mm, vias 0 -> 1
- net Motor2-_t: track 0.00 -> 50.4 mm
- net Motor2+_t: track 0.00 -> 49.3 mm
- net STATE: track 0.00 -> 49.0 mm
- net BAT+: track 0.00 -> 48.0 mm
- net BAT+_Driver: track 0.00 -> 43.0 mm
- net BAT+_t: track 0.00 -> 42.1 mm
- net Button: track 0.00 -> 32.1 mm
- net TXD: track 0.00 -> 32.1 mm
- net RXD: track 0.00 -> 28.5 mm
- net PWMA: track 0.00 -> 22.1 mm
- net Motor1-_t: track 0.00 -> 19.2 mm
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- added copper zone on B.Cu, net GND
- added copper zone on F.Cu, net GND
Other:
- board outline added: 213.3 x 85.2 mm

Commit message: Finished 16 sensor array
Parts:
- removed C9: 22u, Capacitor_SMD:C_0603_1608Metric_Pad1.08x0.95mm_HandSolder
- removed J14, J15: Conn_01x20, Connector_FFC-FPC:Amphenol_F32Q-1A7x1-11020_1x20-1MP_P0.5mm_Horizontal
- added C10: 100n, Capacitor_SMD:C_0603_1608Metric_Pad1.08x0.95mm_HandSolder, F.Cu at (118.8, 68.7)
- added H5: MountingHole, customs:2mm hole, F.Cu at (99.8, 85.1)
- added H6: MountingHole, customs:2mm hole, F.Cu at (121.7, 85.1)
- added J6: Conn_01x20_MountingPin, Connector_FFC-FPC:Amphenol_F32Q-1A7x1-11020_1x20-1MP_P0.5mm_Horizontal, F.Cu at (-20.9, 112.2)
- added J7: Conn_01x20_MountingPin, Connector_FFC-FPC:Amphenol_F32Q-1A7x1-11020_1x20-1MP_P0.5mm_Horizontal, F.Cu at (110.0, 120.5)
- J2: value Conn_01x20 -> Conn_01x20_MountingPin
- moved J2 144.6 mm to (110.0, 89.8)
- moved H3 60.3 mm to (101.9, 97.1)
- moved H4 46.1 mm to (119.7, 97.1)
- moved R89 17.6 mm to (169.4, 98.0), turned to 0 degrees
- moved R20 15.9 mm to (50.1, 100.0)
- moved R83 15.8 mm to (154.9, 77.5), turned to 0 degrees
- moved R38 15.8 mm to (114.9, 63.7), turned to 0 degrees
- moved R91 15.7 mm to (170.9, 107.6)
- moved R86 15.7 mm to (164.1, 88.2), turned to 0 degrees
- moved R43 15.7 mm to (134.9, 68.1)
- moved R44 15.7 mm to (135.1, 70.1), turned to 0 degrees
- moved R78 15.7 mm to (145.2, 72.4), turned to 0 degrees
- moved R37 15.7 mm to (115.0, 61.6)
- moved R85 15.6 mm to (164.1, 86.3)
- moved R92 15.6 mm to (170.9, 109.6), turned to 0 degrees
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Connections:
- J2 pad 10: T9 -> S2_mux
- J2 pad 12: T4 -> S3_mux
- J2 pad 14: T3 -> GND
- J2 pad 16: T2 -> GND
- J2 pad 18: T1 -> GND
- J2 pad 2: T8 -> GND
- J2 pad 4: T7 -> S1_mux
- J2 pad 6: T6 -> S0_mux
- J2 pad 8: T5 -> COM_mux
- J2 pad MP: (no net) -> GND
Routing:
- net +3.3V: track 211.7 -> 598.1 mm, vias 3 -> 22
- net Q16: track 0.00 -> 72.8 mm
- net Q1: track 0.00 -> 71.6 mm
- net Q2: track 0.00 -> 63.2 mm
- net Q15: track 0.00 -> 62.9 mm
- net Q14: track 0.00 -> 53.9 mm
- net Q3: track 0.00 -> 53.7 mm
- net Q13: track 0.00 -> 40.9 mm
- net Q4: track 0.00 -> 40.8 mm
- net Q12: track 0.00 -> 29.4 mm
- net Q5: track 0.00 -> 29.4 mm
- net GND: track 0.00 -> 22.1 mm, vias 0 -> 68
- net Q6: track 0.00 -> 19.8 mm
- net Q11: track 0.00 -> 19.7 mm
- net COM_mux: track 0.00 -> 19.4 mm
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- added copper zone on F.Cu, net +3.3V
Other:
- board size 213.3 x 85.2 mm -> 215.1 x 136.7 mm

Commit message: Start third sensor array
Parts:
- added C1: 100n, Capacitor_SMD:C_0603_1608Metric_Pad1.08x0.95mm_HandSolder, F.Cu at (136.6, 137.8)
- added C2: 100n, Capacitor_SMD:C_0603_1608Metric_Pad1.08x0.95mm_HandSolder, F.Cu at (136.7, 133.1)
- added H10: MountingHole, customs:2mm hole, F.Cu at (120.2, 59.1)
- added H7: MountingHole, customs:2mm hole, F.Cu at (363.2, 129.1)
- added H8: MountingHole, customs:2mm hole, F.Cu at (384.6, 129.1)
- added H9: MountingHole, customs:2mm hole, F.Cu at (98.2, 59.3)
- added J9: Conn_01x20_MountingPin, Connector_FFC-FPC:Amphenol_F32Q-1A7x1-11020_1x20-1MP_P0.5mm_Horizontal, F.Cu at (108.6, 56.5)
- added R1: 10k, Resistor_SMD:R_0603_1608Metric_Pad0.98x0.95mm_HandSolder, F.Cu at (136.6, 139.6)
- added R100: 220, Resistor_SMD:R_0603_1608Metric_Pad0.98x0.95mm_HandSolder, F.Cu at (143.6, 45.8)
- added R101: 220, Resistor_SMD:R_0603_1608Metric_Pad0.98x0.95mm_HandSolder, F.Cu at (113.7, 45.9)
- added R102: 220, Resistor_SMD:R_0603_1608Metric_Pad0.98x0.95mm_HandSolder, F.Cu at (83.6, 45.7)
- added R103: 150, Resistor_SMD:R_0603_1608Metric_Pad0.98x0.95mm_HandSolder, F.Cu at (133.7, 41.7)
- added R104: 150, Resistor_SMD:R_0603_1608Metric_Pad0.98x0.95mm_HandSolder, F.Cu at (103.6, 41.8)
- added R105: 150, Resistor_SMD:R_0603_1608Metric_Pad0.98x0.95mm_HandSolder, F.Cu at (73.6, 41.8)
- added R106: 4k7, Resistor_SMD:R_0603_1608Metric_Pad0.98x0.95mm_HandSolder, F.Cu at (133.7, 43.9)
- added R107: 4k7, Resistor_SMD:R_0603_1608Metric_Pad0.98x0.95mm_HandSolder, F.Cu at (103.6, 44.2)
- added R108: 4k7, Resistor_SMD:R_0603_1608Metric_Pad0.98x0.95mm_HandSolder, F.Cu at (73.6, 43.8)
- added R109: 220, Resistor_SMD:R_0603_1608Metric_Pad0.98x0.95mm_HandSolder, F.Cu at (133.7, 45.8)
- added R110: 220, Resistor_SMD:R_0603_1608Metric_Pad0.98x0.95mm_HandSolder, F.Cu at (103.6, 46.0)
- added R111: 220, Resistor_SMD:R_0603_1608Metric_Pad0.98x0.95mm_HandSolder, F.Cu at (73.6, 45.7)
- added R112: 150, Resistor_SMD:R_0603_1608Metric_Pad0.98x0.95mm_HandSolder, F.Cu at (123.6, 41.7)
- added R113: 150, Resistor_SMD:R_0603_1608Metric_Pad0.98x0.95mm_HandSolder, F.Cu at (93.5, 41.7)
- added R114: 150, Resistor_SMD:R_0603_1608Metric_Pad0.98x0.95mm_HandSolder, F.Cu at (108.6, 26.8)
- added R115: 4k7, Resistor_SMD:R_0603_1608Metric_Pad0.98x0.95mm_HandSolder, F.Cu at (123.7, 43.9)
- added R116: 4k7, Resistor_SMD:R_0603_1608Metric_Pad0.98x0.95mm_HandSolder, F.Cu at (93.6, 43.8)
- added R117: 4k7, Resistor_SMD:R_0603_1608Metric_Pad0.98x0.95mm_HandSolder, F.Cu at (108.7, 29.1)
- added R118: 220, Resistor_SMD:R_0603_1608Metric_Pad0.98x0.95mm_HandSolder, F.Cu at (123.7, 45.8)
- added R119: 220, Resistor_SMD:R_0603_1608Metric_Pad0.98x0.95mm_HandSolder, F.Cu at (93.6, 45.9)
- added R120: 220, Resistor_SMD:R_0603_1608Metric_Pad0.98x0.95mm_HandSolder, F.Cu at (108.6, 30.9)
- added R2: 10k, Resistor_SMD:R_0603_1608Metric_Pad0.98x0.95mm_HandSolder, F.Cu at (136.7, 134.9)
- added R94: 150, Resistor_SMD:R_0603_1608Metric_Pad0.98x0.95mm_HandSolder, F.Cu at (143.5, 41.8)
- added R95: 150, Resistor_SMD:R_0603_1608Metric_Pad0.98x0.95mm_HandSolder, F.Cu at (113.6, 41.8)
- added R96: 150, Resistor_SMD:R_0603_1608Metric_Pad0.98x0.95mm_HandSolder, F.Cu at (83.6, 41.7)
- added R97: 4k7, Resistor_SMD:R_0603_1608Metric_Pad0.98x0.95mm_HandSolder, F.Cu at (143.5, 44.0)
- added R98: 4k7, Resistor_SMD:R_0603_1608Metric_Pad0.98x0.95mm_HandSolder, F.Cu at (113.7, 43.9)
- added R99: 4k7, Resistor_SMD:R_0603_1608Metric_Pad0.98x0.95mm_HandSolder, F.Cu at (83.6, 43.8)
- added SW3: SW_Push, customs:Push button-fp, F.Cu at (142.3, 130.2)
- added U28: QRE1113GR, customs:QRE1113-SMD, B.Cu at (143.6, 43.9)
- added U29: QRE1113GR, customs:QRE1113-SMD, B.Cu at (113.6, 43.9)
- added U30: QRE1113GR, customs:QRE1113-SMD, B.Cu at (83.6, 43.9)
- added U31: QRE1113GR, customs:QRE1113-SMD, B.Cu at (133.6, 43.9)
- added U32: QRE1113GR, customs:QRE1113-SMD, B.Cu at (103.6, 43.9)
- added U33: QRE1113GR, customs:QRE1113-SMD, B.Cu at (73.6, 43.9)
- added U34: QRE1113GR, customs:QRE1113-SMD, B.Cu at (123.6, 43.9)
- added U35: QRE1113GR, customs:QRE1113-SMD, B.Cu at (93.6, 43.9)
- added U36: QRE1113GR, customs:QRE1113-SMD, B.Cu at (108.6, 28.9)
- U19, U2, U20, U4, U5, U6, U7, U8, U9: moved to B.Cu
- moved U2 461.8 mm to (413.2, 112.4), turned to 90 degrees
- moved U4 449.8 mm to (401.7, 112.4), turned to 90 degrees
- moved R50 445.0 mm to (417.2, 114.5), turned to -90 degrees
- moved R49 444.9 mm to (417.2, 110.7), turned to 90 degrees
- moved R51 441.6 mm to (413.5, 118.5), turned to 180 degrees
- moved U5 437.9 mm to (390.3, 112.4), turned to 90 degrees
- moved R53 432.8 mm to (405.7, 114.3), turned to -90 degrees
- moved R52 432.7 mm to (405.6, 110.5), turned to 90 degrees
- moved R54 429.3 mm to (402.0, 118.6), turned to 180 degrees
- moved U6 426.0 mm to (378.9, 112.4), turned to 90 degrees
- moved U20 420.9 mm to (373.2, 97.6), turned to 90 degrees
- moved R56 420.9 mm to (394.3, 114.2), turned to -90 degrees
- moved R55 420.8 mm to (394.3, 110.3), turned to 90 degrees
- moved R57 417.4 mm to (390.7, 118.5), turned to 180 degrees
- moved U7 414.3 mm to (367.4, 112.4), turned to 90 degrees
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Connections:
- net Button renamed Button1
- BlackPill1 pad 31: unconnected-(BlackPill1-PB3-Pad31) -> Button2
- SW2 pad 1: GND -> Net-(C1-Pad1)
Routing:
- net +3.3V: track 598.1 -> 834.6 mm, vias 22 -> 35
- net Button2: track 0.00 -> 57.3 mm
- net T8: track 0.00 -> 39.4 mm
- net T1: track 0.00 -> 38.8 mm
- net N8: track 0.00 -> 34.0 mm
- net T7: track 0.00 -> 29.0 mm
- net T2: track 0.00 -> 28.2 mm
- net N7: track 0.00 -> 24.8 mm
- net T9: track 0.00 -> 19.3 mm
- net GND: track 22.1 -> 41.2 mm, vias 68 -> 80
- net T6: track 0.00 -> 18.8 mm
- net T3: track 0.00 -> 18.0 mm
- net N6: track 0.00 -> 15.5 mm
- net N4: track 0.00 -> 9.93 mm
- net N5: track 0.00 -> 8.80 mm
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Other:
- board size 215.1 x 136.7 mm -> 389.6 x 177.9 mm

Commit message: Start custom sensor array
Parts:
- moved C10 289.2 mm to (93.1, 27.8)
- moved H3 289.2 mm to (74.5, 51.8)
- moved H4 289.2 mm to (95.9, 51.8)
- moved H5 289.2 mm to (74.2, 44.2)
- moved H6 289.2 mm to (96.1, 44.2)
- moved H7 289.2 mm to (74.1, 129.4)
- moved H8 289.2 mm to (95.5, 129.4)
- moved J2 289.2 mm to (84.4, 48.9)
- moved J6 289.2 mm to (84.0, 127.4)
- moved R19 289.2 mm to (23.5, 70.6)
- moved R20 289.2 mm to (24.5, 59.1)
- moved R21 289.2 mm to (30.5, 49.3)
- moved R22 289.2 mm to (23.3, 66.6)
- moved R23 289.2 mm to (24.4, 55.3)
- moved R24 289.2 mm to (23.5, 68.6)
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Routing:
- net +3.3V: track 834.6 -> 1001.7 mm, vias 35 -> 41
- net GND: track 41.2 -> 87.2 mm, vias 80 -> 82
- net N1: track 0.00 -> 36.5 mm
- net N2: track 0.00 -> 27.8 mm
- net N9: track 0.00 -> 23.2 mm
- net N3: track 0.00 -> 19.1 mm
- net Net-(R83-Pad1): track 2.30 -> 5.35 mm
- net Motor1+_t: track 16.4 -> 18.1 mm
- net N6: track 15.5 -> 16.5 mm
Other:
- board size 389.6 x 177.9 mm -> 262.1 x 172.5 mm
- board text added: "Battery Kill"
- board text added: "MP1584"
- board text added: "Motor Kill"
- board text added: "TB6612"
