File: Lavender 1.0/customssensor.kicad_sch (KiCad schematic)
At the start: 45 parts, among them Q1 BPW40, Q2 BPW40, Q3 BPW40, Q4 BPW40, Q5 BPW40, Q6 BPW40, Q7 BPW40, Q8 BPW40, Q9 BPW40

Commit message: Finished PCB
Parts:
- D1, D2, D3, D4, D5, D6, D7, D8, D9: footprint (none) -> LED_THT:LED_D5.0mm_Clear
- Q1: footprint LED_THT:LED_D5.0mm_Horizontal_O6.35mm_Z3.0mm -> LED_THT:LED_D5.0mm_Clear
Connections:
- net T1 renamed L1
- net T2 renamed L2
- net T3 renamed L3
- net T4 renamed L4
- net T5 renamed L5
- net T6 renamed L6
- net T7 renamed L7
- net T8 renamed L8
- net T9 renamed L9
Changed lines of the file:
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@@
 		)
 	)
-	(global_label "T2"
+	(global_label "L2"
 		(shape output)
 		(at 177.8 38.1 0)
@@
 		)
 		(property "Intersheetrefs" "${INTERSHEET_REFS}"
-			(at 182.9623 38.1 0)
+			(at 183.0228 38.1 0)
 			(hide yes)
 			(show_name no)
@@
 		)
 	)
-	(global_label "T4"
+	(global_label "L4"
 		(shape output)
 		(at 138.43 63.5 0)
@@
 		)
 		(property "Intersheetrefs" "${INTERSHEET_REFS}"
-			(at 143.5923 63.5 0)
+			(at 143.6528 63.5 0)
 			(hide yes)
 			(show_name no)
@@
 		)
 	)
-	(global_label "T5"
+	(global_label "L5"
 		(shape output)
 		(at 177.8 62.23 0)
@@
 		)
 		(property "Intersheetrefs" "${INTERSHEET_REFS}"
-			(at 182.9623 62.23 0)
+			(at 183.0228 62.23 0)
 			(hide yes)
 			(show_name no)
@@
 		)
 	)
-	(global_label "T9"
+	(global_label "L9"
 		(shape output)
 		(at 217.17 88.9 0)
@@
 		)
 		(property "Intersheetrefs" "${INTERSHEET_REFS}"
-			(at 222.3323 88.9 0)
+			(at 222.3928 88.9 0)
 			(hide yes)
 			(show_name no)
@@
 		)
 	)
-	(global_label "T6"
+	(global_label "L6"
 		(shape output)
 		(at 217.17 60.96 0)
@@
 		)
 		(property "Intersheetrefs" "${INTERSHEET_REFS}"
-			(at 222.3323 60.96 0)
+			(at 222.3928 60.96 0)
 			(hide yes)
 			(show_name no)
@@
 		)
 	)
-	(global_label "T1"
+	(global_label "L1"
 		(shape output)
 		(at 138.43 39.37 0)
@@
 		)
 		(property "Intersheetrefs" "${INTERSHEET_REFS}"
-			(at 143.5923 39.37 0)
+			(at 143.6528 39.37 0)
 			(hide yes)
 			(show_name no)
@@
 		)
 	)
-	(global_label "T8"
+	(global_label "L8"
 		(shape output)
 		(at 177.8 90.17 0)
@@
 		)
 		(property "Intersheetrefs" "${INTERSHEET_REFS}"
-			(at 182.9623 90.17 0)
+			(at 183.0228 90.17 0)
 			(hide yes)
 			(show_name no)
@@
 		)
 	)
-	(global_label "T7"
+	(global_label "L7"
 		(shape output)
 		(at 138.43 91.44 0)
@@
 		)
 		(property "Intersheetrefs" "${INTERSHEET_REFS}"
-			(at 143.5923 91.44 0)
+			(at 143.6528 91.44 0)
 			(hide yes)
 			(show_name no)
@@
 		)
 	)
-	(global_label "T3"
+	(global_label "L3"
 		(shape output)
 		(at 217.17 36.83 0)
@@
 		)
 		(property "Intersheetrefs" "${INTERSHEET_REFS}"
-			(at 222.3323 36.83 0)
+			(at 222.3928 36.83 0)
 			(hide yes)
 			(show_name no)
@@
 			)
 		)
-		(property "Footprint" ""
+		(property "Footprint" "LED_THT:LED_D5.0mm_Clear"
 			(at 58.42 52.07 0)
 			(hide yes)
@@
 			)
 		)
-		(property "Footprint" ""
+		(property "Footprint" "LED_THT:LED_D5.0mm_Clear"
 			(at 34.29 52.07 0)
 			(hide yes)
@@
 			)
 		)
-		(property "Footprint" ""
+		(property "Footprint" "LED_THT:LED_D5.0mm_Clear"
 			(at 82.55 53.34 0)
 			(hide yes)
@@
 			)
 		)
-		(property "Footprint" ""
+		(property "Footprint" "LED_THT:LED_D5.0mm_Clear"
 			(at 58.42 35.56 0)
 			(hide yes)
@@
 			)
 		)
-		(property "Footprint" ""
+		(property "Footprint" "LED_THT:LED_D5.0mm_Clear"
 			(at 58.42 68.58 0)
 			(hide yes)
@@
 			)
 		)
-		(property "Footprint" ""
+		(property "Footprint" "LED_THT:LED_D5.0mm_Clear"
 			(at 34.29 68.58 0)
 			(hide yes)
@@
 			)
 		)
-		(property "Footprint" "LED_THT:LED_D5.0mm_Horizontal_O6.35mm_Z3.0mm"
+		(property "Footprint" "LED_THT:LED_D5.0mm_Clear"
 			(at 118.364 49.022 0)
 			(hide yes)
@@
 			)
 		)
-		(property "Footprint" ""
+		(property "Footprint" "LED_THT:LED_D5.0mm_Clear"
 			(at 82.55 68.58 0)
 			(hide yes)
@@
 			)
 		)
-		(property "Footprint" ""
+		(property "Footprint" "LED_THT:LED_D5.0mm_Clear"
 			(at 82.55 35.56 0)
 			(hide yes)
@@
 			)
 		)
-		(property "Footprint" ""
+		(property "Footprint" "LED_THT:LED_D5.0mm_Clear"
 			(at 34.29 35.56 0)
 			(hide yes)
