File: Lavender 1.0/line follower simple.kicad_sch (KiCad schematic)
At the start: 36 parts, among them J1 XT30UPB-M, J14 Conn_01x20_MountingPin, J2 Conn_01x20_MountingPin, J3 Conn_01x02_Pin, J4 Conn_01x02_Pin, J6 Conn_01x20_MountingPin, J7 Conn_01x20_MountingPin, J9 Conn_01x20_MountingPin, SW2 SW_Push, SW3 SW_Push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

Commit message: Finished PCB
Connections:
- net T1: no longer J14.18 (Pin_18)
- net T2: no longer J14.16 (Pin_16)
- net T3: no longer J14.14 (Pin_14)
- net T4: no longer J14.12 (Pin_12)
- net T5: no longer J14.8 (Pin_8)
- net T6: no longer J14.6 (Pin_6)
- net T7: no longer J14.4 (Pin_4)
- net T8: no longer J14.2 (Pin_2)
- net T9: no longer J14.10 (Pin_10)
- new net L1: J14.18 (Pin_18)
- new net L2: J14.16 (Pin_16)
- new net L3: J14.14 (Pin_14)
- new net L4: J14.12 (Pin_12)
- new net L5: J14.8 (Pin_8)
- new net L6: J14.6 (Pin_6)
- new net L7: J14.4 (Pin_4)
- new net L8: J14.2 (Pin_2)
- new net L9: J14.10 (Pin_10)
