File: old/flf.kicad_sch (KiCad schematic)
At the start: 70 parts, among them IC1 TB6612FNG, J1 Conn_01x04_Pin, J2 XT30UPB-M, J3 Conn_01x02_Socket, J4 Conn_01x02_Socket, U1 STM32F411CEUx, U10 QRE1113GR, U11 QRE1113GR, U2 TCRT5000L, U3 QRE1113GR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

Commit message: new
Parts:
- removed J1: Conn_01x04_Pin, symbol Connector:Conn_01x04_Pin
- removed J2: XT30UPB-M, XT30UPB-M:AMASS_XT30UPB-M, symbol customs:XT30UPB-M
- added J1: XT60-M, XT60-M:AMASS_XT60-M, symbol New_Library:XT60-M
- added J5: Conn_01x05_Pin, symbol Connector:Conn_01x05_Pin
Connections:
- net +3.3V: now also J5.1 (Pin_1)
- net BAT+: now also J1.P (POS)
- net BAT-: no longer MP1. (IN+)
- net GND: now also J1.N (NEG), J5.4 (Pin_4)
- net SWCLK: now also J5.3 (Pin_3)
- net SWDIO: now also J5.2 (Pin_2)
- new net SWDO: J5.5 (Pin_5)

Commit message: Curved array for tcrt500
Parts:
- removed C5: 100n, symbol Device:C
- removed FB1: FerriteBead_Small, symbol Device:FerriteBead_Small
- removed R7, R8: 10k, symbol Device:R
- removed U2: TCRT5000L, TCRT5000L:XDCR_TCRT5000L, symbol customs:TCRT5000L
- added C24, C25, C26, C5: C_Small, symbol Device:C_Small
- added D2: LED, symbol Device:LED
- added L1: L, symbol Device:L
- added R24: 1k, symbol Device:R
- added R7, R8: R_Small, symbol Device:R_Small
- added SW1, SW2: SW_Push, symbol Switch:SW_Push
- M1, M2, MM1, MM2, MP1: value ~ -> (none)
Connections:
- net +3.3V: now also C25.1, D2.2 (A), L1.2, R7.1, SW2.2
- net GND: now also C24.2, C25.2, C26.1, C5.2, R24.2, R8.1, SW1.2
- net VDDA: now also C24.1, L1.1
- net Pull D renamed BOOT
- net BOOT: now also C26.2, R8.2, SW2.1
- net Pull U renamed NRST
- net NRST: now also C5.1, R7.2, SW1.1
- new net: D2.1 (K), R24.1
Other:
- note added: "Boot button"
- note added: "PC13 LED"
- note added: "Power LED"
- note added: "Reset button"
- moved on the sheet: C13, C8, D1, J1, MP1, R1, R5, R6
