File: Lavender 1.0 (Blackpill vers)/line follower simple.kicad_pcb (KiCad board)
At the start: 2 copper layers, 214 x 187.9 mm, 259 parts, among them J1 XT30UPB-M, J10 Conn_01x13_Pin, J11 Conn_01x13_Pin, J12 Conn_01x13_Pin, J13 Conn_01x13_Pin, J14 Conn_01x20_MountingPin, J15 Conn_01x11_Pin, J16 Conn_01x11_Pin, J17 Conn_01x11_Pin, J18 Conn_01x11_Pin, J19 Conn_01x11_Pin, J2 Conn_01x20_MountingPin, J3 Conn_01x02_Pin, J4 Conn_01x02_Pin, J5 Conn_01x28_Pin, J6 Conn_01x20_MountingPin, J7 Conn_01x20_MountingPin, J8 Conn_01x28_Pin, J9 Conn_01x20_MountingPin, Q1 BPW40, Q2 BPW40, Q3 BPW40, Q4 BPW40, Q5 BPW40, Q6 BPW40, Q7 BPW40, Q8 BPW40, Q9 BPW40, SW2 SW_Push, SW3 SW_Push, SW5 SW_Push_DPDT, SW6 SW_Push_DPDT, U1 74HC4067, U10 QRE1113GR, U11 QRE1113GR, U12 QRE1113GR, U13 QRE1113GR, U14 QRE1113GR, U15 QRE1113GR, U16 QRE1113GR, U17 QRE1113GR, U18 QRE1113GR, U19 TCRT5000L, U2 TCRT5000L, U20 TCRT5000L, U21 QRE1113GR, U22 QRE1113GR, U23 QRE1113GR, U24 QRE1113GR, U25 QRE1113GR, U26 QRE1113GR, U27 QRE1113GR, U28 QRE1113GR, U29 QRE1113GR, U30 QRE1113GR, U31 QRE1113GR, U32 QRE1113GR, U33 QRE1113GR, U34 QRE1113GR, U35 QRE1113GR, U36 QRE1113GR, U4 TCRT5000L, U5 TCRT5000L, U6 TCRT5000L, U7 TCRT5000L, U8 TCRT5000L, U9 TCRT5000L

Commit message: Silkscreen fixes
Other:
- board text added: "3.3V IN"
- board text added: "3.3V OUT"
- board text added: "BAT IN"
- board text added: "MOTOR 1+"
- board text added: "MOTOR 1-"
- board text added: "MOTOR 2+"
- board text added: "MOTOR 2-"
Changed lines of the file:
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@@
+		)
+	)
+	(gr_text "GND"
+		(at 171.8 101.25 0)
+		(layer "B.SilkS")
+		(effects
+			(font
+				(size 0.6 0.6)
+				(thickness 0.1)
+			)
+			(justify left bottom mirror)
+		)
+	)
+	(gr_text "GND"
+		(at 172.1 88.35 0)
+		(layer "B.SilkS")
+		(effects
+			(font
+				(size 0.6 0.6)
+				(thickness 0.1)
+			)
+			(justify left bottom mirror)
+		)
+	)
+	(gr_text "BAT IN"
+		(at 172.75 83.3 0)
+		(layer "B.SilkS")
+		(effects
+			(font
+				(size 0.6 0.6)
+				(thickness 0.1)
+			)
+			(justify left bottom mirror)
+		)
+	)
+	(gr_text "3.3V IN"
+		(at 173.05 85.8 0)
+		(layer "B.SilkS")
+		(effects
+			(font
+				(size 0.6 0.6)
+				(thickness 0.1)
+			)
+			(justify left bottom mirror)
+		)
+	)
+	(gr_text "MOTOR 1+"
+		(at 174.1 90.95 0)
+		(layer "B.SilkS")
+		(effects
+			(font
+				(size 0.6 0.6)
+				(thickness 0.1)
+			)
+			(justify left bottom mirror)
+		)
+	)
+	(gr_text "MOTOR 2-"
+		(at 174.1 96.116667 0)
+		(layer "B.SilkS")
+		(effects
+			(font
+				(size 0.6 0.6)
+				(thickness 0.1)
+			)
+			(justify left bottom mirror)
+		)
+	)
+	(gr_text "MOTOR 1-"
+		(at 174.15 93.533333 0)
+		(layer "B.SilkS")
+		(effects
+			(font
+				(size 0.6 0.6)
+				(thickness 0.1)
+			)
+			(justify left bottom mirror)
+		)
+	)
+	(gr_text "MOTOR 2+"
+		(at 174.15 98.7 0)
+		(layer "B.SilkS")
+		(effects
+			(font
+				(size 0.6 0.6)
+				(thickness 0.1)
+			)
+			(justify left bottom mirror)
+		)
+	)
+	(gr_text "GND"
+		(at 179.3 101.3 0)
+		(layer "B.SilkS")
+		(effects
+			(font
+				(size 0.6 0.6)
+				(thickness 0.1)
+			)
+			(justify left bottom mirror)
+		)
+	)
+	(gr_text "3.3V IN"
+		(at 179.7 91.05 0)
+		(layer "B.SilkS")
+		(effects
+			(font
+				(size 0.6 0.6)
+				(thickness 0.1)
+			)
+			(justify left bottom mirror)
 		)
 	)
@@
 		(layer "B.SilkS")
 		(effects
+			(font
+				(size 1 1)
+				(thickness 0.1)
+			)
+			(justify left bottom mirror)
+		)
+	)
+	(gr_text "3.3V OUT"
+		(at 167.55 134.3 270)
+		(layer "B.SilkS")
+		(effects
+			(font
+				(size 1 1)
+				(thickness 0.1)
+			)
+			(justify left bottom mirror)
+		)
+	)
+	(gr_text "BAT IN"
+		(at 167.75 118.4 270)
+		(layer "B.SilkS")
+		(effects
