File: Lavender 1.0 (Blackpill vers)/QRE1113.kicad_sch (KiCad schematic)
At the start: 100 parts, among them U10 QRE1113GR, U11 QRE1113GR, U12 QRE1113GR, U13 QRE1113GR, U14 QRE1113GR, U15 QRE1113GR, U16 QRE1113GR, U17 QRE1113GR, U18 QRE1113GR, U21 QRE1113GR, U22 QRE1113GR, U23 QRE1113GR, U24 QRE1113GR, U25 QRE1113GR, U26 QRE1113GR, U27 QRE1113GR, U28 QRE1113GR, U29 QRE1113GR, U30 QRE1113GR, U31 QRE1113GR, U32 QRE1113GR, U33 QRE1113GR, U34 QRE1113GR, U35 QRE1113GR, U36 QRE1113GR

Commit message: fix footprint
Parts:
- U10, U11, U12, U13, U14, U15, U16, U17, U18, U21, U22, U23, U24, U25, U26, U27, U28, U29, U30, U31, U32, U33, U34, U35, U36: footprint customs:QRE1113-SMD -> MyCustoms:QRE1113-SMD
Changed lines of the file:
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@@
 			)
 		)
-		(property "Footprint" "customs:QRE1113-SMD"
+		(property "Footprint" "MyCustoms:QRE1113-SMD"
 			(at 256.54 29.21 0)
 			(hide yes)
@@
 			)
 		)
-		(property "Footprint" "customs:QRE1113-SMD"
+		(property "Footprint" "MyCustoms:QRE1113-SMD"
 			(at 184.15 62.23 0)
 			(hide yes)
@@
 			)
 		)
-		(property "Footprint" "customs:QRE1113-SMD"
+		(property "Footprint" "MyCustoms:QRE1113-SMD"
 			(at 218.44 29.21 0)
 			(hide yes)
@@
 			)
 		)
-		(property "Footprint" "customs:QRE1113-SMD"
+		(property "Footprint" "MyCustoms:QRE1113-SMD"
 			(at 256.54 62.23 0)
 			(hide yes)
@@
 			)
 		)
-		(property "Footprint" "customs:QRE1113-SMD"
+		(property "Footprint" "MyCustoms:QRE1113-SMD"
 			(at 68.58 101.6 0)
 			(hide yes)
@@
 			)
 		)
-		(property "Footprint" "customs:QRE1113-SMD"
+		(property "Footprint" "MyCustoms:QRE1113-SMD"
 			(at 256.54 96.52 0)
 			(hide yes)
@@
 			)
 		)
-		(property "Footprint" "customs:QRE1113-SMD"
+		(property "Footprint" "MyCustoms:QRE1113-SMD"
 			(at 218.44 62.23 0)
 			(hide yes)
@@
 			)
 		)
-		(property "Footprint" "customs:QRE1113-SMD"
+		(property "Footprint" "MyCustoms:QRE1113-SMD"
 			(at 219.71 129.54 0)
 			(hide yes)
@@
 			)
 		)
-		(property "Footprint" "customs:QRE1113-SMD"
+		(property "Footprint" "MyCustoms:QRE1113-SMD"
 			(at 102.87 101.6 0)
 			(hide yes)
@@
 			)
 		)
-		(property "Footprint" "customs:QRE1113-SMD"
+		(property "Footprint" "MyCustoms:QRE1113-SMD"
 			(at 257.81 129.54 0)
 			(hide yes)
@@
 			)
 		)
-		(property "Footprint" "customs:QRE1113-SMD"
+		(property "Footprint" "MyCustoms:QRE1113-SMD"
 			(at 33.02 34.29 0)
 			(hide yes)
@@
 			)
 		)
-		(property "Footprint" "customs:QRE1113-SMD"
+		(property "Footprint" "MyCustoms:QRE1113-SMD"
 			(at 68.58 67.31 0)
 			(hide yes)
@@
 			)
 		)
-		(property "Footprint" "customs:QRE1113-SMD"
+		(property "Footprint" "MyCustoms:QRE1113-SMD"
 			(at 33.02 101.6 0)
 			(hide yes)
@@
 			)
 		)
-		(property "Footprint" "customs:QRE1113-SMD"
+		(property "Footprint" "MyCustoms:QRE1113-SMD"
 			(at 102.87 67.31 0)
 			(hide yes)
@@
 			)
 		)
-		(property "Footprint" "customs:QRE1113-SMD"
+		(property "Footprint" "MyCustoms:QRE1113-SMD"
 			(at 218.44 96.52 0)
 			(hide yes)
@@
 			)
 		)
-		(property "Footprint" "customs:QRE1113-SMD"
+		(property "Footprint" "MyCustoms:QRE1113-SMD"
 			(at 68.58 34.29 0)
 			(hide yes)
@@
 			)
 		)
-		(property "Footprint" "customs:QRE1113-SMD"
+		(property "Footprint" "MyCustoms:QRE1113-SMD"
 			(at 102.87 34.29 0)
 			(hide yes)
@@
 			)
 		)
-		(property "Footprint" "customs:QRE1113-SMD"
+		(property "Footprint" "MyCustoms:QRE1113-SMD"
 			(at 148.59 29.21 0)
 			(hide yes)
@@
 			)
 		)
-		(property "Footprint" "customs:QRE1113-SMD"
+		(property "Footprint" "MyCustoms:QRE1113-SMD"
 			(at 148.59 62.23 0)
 			(hide yes)
@@
 			)
 		)
-		(property "Footprint" "customs:QRE1113-SMD"
+		(property "Footprint" "MyCustoms:QRE1113-SMD"
 			(at 184.15 96.52 0)
 			(hide yes)
@@
 			)
 		)
-		(property "Footprint" "customs:QRE1113-SMD"
+		(property "Footprint" "MyCustoms:QRE1113-SMD"
 			(at 33.02 67.31 0)
 			(hide yes)
@@
 			)
 		)
-		(property "Footprint" "customs:QRE1113-SMD"
+		(property "Footprint" "MyCustoms:QRE1113-SMD"
 			(at 148.59 96.52 0)
 			(hide yes)
@@
 			)
 		)
-		(property "Footprint" "customs:QRE1113-SMD"
+		(property "Footprint" "MyCustoms:QRE1113-SMD"
 			(at 184.15 29.21 0)
 			(hide yes)
@@
 			)
 		)
-		(property "Footprint" "customs:QRE1113-SMD"
+		(property "Footprint" "MyCustoms:QRE1113-SMD"
 			(at 149.86 129.54 0)
 			(hide yes)
@@
 			)
 		)
-		(property "Footprint" "customs:QRE1113-SMD"
+		(property "Footprint" "MyCustoms:QRE1113-SMD"
 			(at 185.42 129.54 0)
 			(hide yes)
