File: Lavender 1.0 (Blackpill vers)/TCRT_sensors.kicad_sch (KiCad schematic)
At the start: 36 parts, among them U19 TCRT5000L, U2 TCRT5000L, U20 TCRT5000L, U4 TCRT5000L, U5 TCRT5000L, U6 TCRT5000L, U7 TCRT5000L, U8 TCRT5000L, U9 TCRT5000L

Commit message: fix footprint
Parts:
- U19, U2, U20, U4, U5, U6, U7, U8, U9: footprint customs:XDCR_TCRT5000L -> MyCustoms:XDCR_TCRT5000L
Changed lines of the file:
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@@
 			)
 		)
-		(property "Footprint" "customs:XDCR_TCRT5000L"
+		(property "Footprint" "MyCustoms:XDCR_TCRT5000L"
 			(at 105.41 80.01 0)
 			(hide yes)
@@
 			)
 		)
-		(property "Footprint" "customs:XDCR_TCRT5000L"
+		(property "Footprint" "MyCustoms:XDCR_TCRT5000L"
 			(at 69.85 80.01 0)
 			(hide yes)
@@
 			)
 		)
-		(property "Footprint" "customs:XDCR_TCRT5000L"
+		(property "Footprint" "MyCustoms:XDCR_TCRT5000L"
 			(at 68.58 115.57 0)
 			(hide yes)
@@
 			)
 		)
-		(property "Footprint" "customs:XDCR_TCRT5000L"
+		(property "Footprint" "MyCustoms:XDCR_TCRT5000L"
 			(at 71.12 45.72 0)
 			(hide yes)
@@
 			)
 		)
-		(property "Footprint" "customs:XDCR_TCRT5000L"
+		(property "Footprint" "MyCustoms:XDCR_TCRT5000L"
 			(at 34.29 80.01 0)
 			(hide yes)
@@
 			)
 		)
-		(property "Footprint" "customs:XDCR_TCRT5000L"
+		(property "Footprint" "MyCustoms:XDCR_TCRT5000L"
 			(at 104.14 115.57 0)
 			(hide yes)
@@
 			)
 		)
-		(property "Footprint" "customs:XDCR_TCRT5000L"
+		(property "Footprint" "MyCustoms:XDCR_TCRT5000L"
 			(at 33.02 115.57 0)
 			(hide yes)
@@
 			)
 		)
-		(property "Footprint" "customs:XDCR_TCRT5000L"
+		(property "Footprint" "MyCustoms:XDCR_TCRT5000L"
 			(at 106.68 45.72 0)
 			(hide yes)
@@
 			)
 		)
-		(property "Footprint" "customs:XDCR_TCRT5000L"
+		(property "Footprint" "MyCustoms:XDCR_TCRT5000L"
 			(at 35.56 45.72 0)
 			(hide yes)
